File: CanoKey Nano-A v1.1/PCB/Main.sch (KiCad schematic (older format))
At the start: 23 parts, among them J1 USB_A_PCB, U2 USBLC6-2SC6, U3 STM32L432KCUx, U4 AP7331-33SNG-7

Commit message: compact PCB
Parts:
- removed C2: 100n, Capacitor_SMD:C_0603_1608Metric, symbol Device:C_Small
- removed D?: LED_R, Diode_SMD:D_0805_2012Metric, symbol Device:LED_Small
- removed R3: 2.2k, Resistor_SMD:R_0603_1608Metric, symbol Device:R_Small
- removed TP1, TP5: TestPoint, TestPoint:TestPoint_Pad_D1.0mm, symbol Connector:TestPoint
- removed TP4: TestPoint, TestPoint:TestPoint_Pad_D4.0mm, symbol Connector:TestPoint
- gave numbers to parts that had none: 1
Connections:
- net DBG_TX: no longer names the net of U3.8 (PA2)
- net LEDR: no longer names the net of U3.15 (PB1)
- net RST: no longer names the net of U3.4 (NRST)
Changed lines of the file:
@@
-$EndComp
-$Comp
-L Connector:TestPoint TP1
-U 1 1 5EF09477
-P 8850 3600
-F 0 "TP1" H 8908 3718 50  0000 L CNN
-F 1 "TestPoint" H 8908 3627 50  0001 L CNN
-F 2 "TestPoint:TestPoint_Pad_D1.0mm" H 9050 3600 50  0001 C CNN
-F 3 "~" H 9050 3600 50  0001 C CNN
-	1    8850 3600
-	1    0    0    -1
 $EndComp
 $Comp
@@
 	0    1    -1   0
 $EndComp
-Text Label 5150 2000 0    50   ~ 0
-RST
 Text Label 6850 2000 2    50   ~ 0
 IRQN
 Text Label 6850 2100 2    50   ~ 0
 V_RF
-Text Label 6850 2200 2    50   ~ 0
-DBG_TX
 Text Label 6850 2400 2    50   ~ 0
 SSN
@@
 Text Label 6850 3200 2    50   ~ 0
 USB_P
-Text Label 5150 3000 0    50   ~ 0
-LEDR
 Wire Wire Line
 	6100 1800 6100 1700
@@
 	6000 3800 6000 3900
 Wire Wire Line
-	5150 2000 5500 2000
-Wire Wire Line
 	5150 2400 5500 2400
 Wire Wire Line
 	5150 3100 5500 3100
 Wire Wire Line
-	5150 3000 5500 3000
-Wire Wire Line
 	6500 3400 6850 3400
 Wire Wire Line
@@
 	6500 2400 6850 2400
 Wire Wire Line
-	6500 2200 6850 2200
-Wire Wire Line
 	6500 2100 6850 2100
 Wire Wire Line
 	6500 2000 6850 2000
-Text Label 8500 3700 0    50   ~ 0
-DBG_TX
-Wire Wire Line
-	8850 3700 8500 3700
 Text Label 8500 3900 0    50   ~ 0
 SWCLK
@@
 $EndComp
 Wire Wire Line
-	8850 3700 8850 3600
-Wire Wire Line
 	9150 3800 9150 3600
 Wire Wire Line
@@
 Wire Wire Line
 	3050 6250 3400 6250
-$Comp
-L Device:R_Small R3
-U 1 1 5F013A5D
-P 6350 6100
-F 0 "R3" V 6400 6200 50  0000 L CNN
-F 1 "2.2k" H 6409 6055 50  0000 L CNN
-F 2 "Resistor_SMD:R_0603_1608Metric" H 6350 6100 50  0001 C CNN
-F 3 "~" H 6350 6100 50  0001 C CNN
-F 4 "C4190" H 6350 6100 50  0001 C CNN "LCSC"
-F 5 "5%" H 6350 6100 50  0001 C CNN "Tolerance"
-	1    6350 6100
-	-1   0    0    -1
-$EndComp
-Wire Wire Line
-	6350 5900 6350 6000
 $Comp
 L Device:R_Small R7
@@
 	1    0    0    -1
 $EndComp
-Wire Wire Line
-	6550 6200 6550 6300
-Wire Wire Line
-	6350 6300 6350 6200
-Wire Wire Line
-	6350 6300 6550 6300
-Connection ~ 6550 6300
-Wire Wire Line
-	6550 6300 6550 6400
 $Comp
 L Device:R_Small R5
@@
 $EndComp
 $Comp
-L Device:C_Small C2
-U 1 1 5F0BC63B
-P 3000 1700
-F 0 "C2" H 3092 1746 50  0000 L CNN
-F 1 "100n" H 3092 1655 50  0000 L CNN
-F 2 "Capacitor_SMD:C_0603_1608Metric" H 3000 1700 50  0001 C CNN
-F 3 "~" H 3000 1700 50  0001 C CNN
-F 4 "C14663" H 3000 1700 50  0001 C CNN "LCSC"
-F 5 "50v" H 3000 1700 50  0001 C CNN "Voltage"
-F 6 "x7r" H 3000 1700 50  0001 C CNN "Dielectric"
-	1    3000 1700
-	1    0    0    -1
-$EndComp
-$Comp
 L power:+3.3V #PWR0108
 U 1 1 5F0C4708
@@
 	1    0    0    -1
 $EndComp
-Wire Wire Line
-	3400 1400 3400 1500
-Wire Wire Line
-	3400 1600 3400 1500
-Wire Wire Line
-	3400 1500 3000 1500
-Wire Wire Line
-	3000 1500 3000 1600
-Connection ~ 3400 1500
-Wire Wire Line
-	3400 2000 3400 1900
-Wire Wire Line
-	3400 1800 3400 1900
-Wire Wire Line
-	3400 1900 3000 1900
-Wire Wire Line
-	3000 1900 3000 1800
-Connection ~ 3400 1900
 $Comp
 L power:GND #PWR0109
@@
 $EndComp
 $Comp
-L Connector:TestPoint TP4
-U 1 1 5F22D5EF
-P 10500 1500
-F 0 "TP4" H 10558 1618 50  0000 L CNN
-F 1 "TestPoint" H 10558 1527 50  0001 L CNN
-F 2 "TestPoint:TestPoint_Pad_D4.0mm" H 10700 1500 50  0001 C CNN
-F 3 "~" H 10700 1500 50  0001 C CNN
-	1    10500 1500
-	0    1    1    0
-$EndComp
-$Comp
 L Device:R_Small R1
 U 1 1 5F23DD6E
@@
 	10050 1650 10050 1500
 Wire Wire Line
-	10050 1500 10500 1500
+	10050 1500 10650 1500
 Connection ~ 10050 1500
 $Comp
@@
 Wire Wire Line
 	1700 7250 2300 7250
-Text Label 8500 4000 0    50   ~ 0
-RST
-$Comp
-L Connector:TestPoint TP5
-U 1 1 5F373F27
-P 9750 3600
-F 0 "TP5" H 9808 3718 50  0000 L CNN
-F 1 "TestPoint" H 9808 3627 50  0001 L CNN
-F 2 "TestPoint:TestPoint_Pad_D1.0mm" H 9950 3600 50  0001 C CNN
-F 3 "~" H 9950 3600 50  0001 C CNN
-	1    9750 3600
-	1    0    0    -1
-$EndComp
-Wire Wire Line
-	8500 4000 9750 4000
-Wire Wire Line
-	9750 3600 9750 4000
-Text Label 5500 5900 0    50   ~ 0
-LEDR
 Text Label 5500 5700 0    50   ~ 0
 LEDG
@@
 	5150 3300 5500 3300
 $Comp
-L Device:LED_Small D?
+L Device:LED_Small D1
 U 1 1 5F76BCE4
 P 6050 5700
-F 0 "D?" H 6050 5935 50  0000 C CNN
+F 0 "D1" H 6050 5935 50  0000 C CNN
 F 1 "LED_G" H 6050 5844 50  0000 C CNN
 F 2 "Diode_SMD:D_0805_2012Metric" V 6050 5700 50  0001 C CNN
@@
 	-1   0    0    -1
 $EndComp
-$Comp
-L Device:LED_Small D?
-U 1 1 5F76C9EB
-P 6050 5900
-F 0 "D?" H 6050 6135 50  0000 C CNN
-F 1 "LED_R" H 6050 6044 50  0000 C CNN
-F 2 "Diode_SMD:D_0805_2012Metric" V 6050 5900 50  0001 C CNN
-F 3 "~" V 6050 5900 50  0001 C CNN
-F 4 "" H 6050 5900 50  0001 C CNN "LCSC"
-	1    6050 5900
-	-1   0    0    1
-$EndComp
-Wire Wire Line
-	5500 5900 5950 5900
-Wire Wire Line
-	6150 5900 6350 5900
 Wire Wire Line
 	6150 5700 6550 5700
@@
 Wire Wire Line
 	5500 3500 5150 3500
+Wire Wire Line
+	6550 6200 6550 6400
+Wire Wire Line
+	3400 1400 3400 1600
+Wire Wire Line
+	3400 1800 3400 2000
+Wire Wire Line
+	10650 1500 10650 1600
+Wire Wire Line
+	10650 1600 10850 1600
+Wire Wire Line
+	10850 1600 10850 1400
+Wire Wire Line
+	10850 1400 10650 1400
+Wire Wire Line
+	10650 1400 10650 1500
+Connection ~ 10650 1500
 $EndSCHEMATC
